File: energyReplay/Control.kicad_sch (KiCad schematic)
At the start: 24 parts, among them J1 Conn_02x07_Odd_Even, J2 Power Select, J3 Conn_01x02_Pin, J4 Conn_01x02_Pin, J5 Conn_02x10_Counter_Clockwise, SW1 SW_Push, SW2 SW_Push, U1 MSP430FR5994IPN

Commit message: 1.1 KiCAD project
Parts:
- added C11, C12: 100n, Capacitor_SMD:C_1206_3216Metric, symbol Device:C_Small
- added NT1, NT2, NT3, NT4: NetTie_2, NetTie-0.2mm:NetTie-2_SMD_Pad0.2mm, symbol Device:NetTie_2
- added Y1: Crystal, MS1V-T1K:XTAL_MS1V-T1K-32.768KHZ-12.5PF-20PPM-TA-QC, symbol Device:Crystal
Connections:
- net GND: now also J5.12 (Pin_12), J5.13 (Pin_13), J5.14 (Pin_14); no longer U1.76 (AVSS2), U1.79 (AVSS1)
- net at U1.77 (PJ.4_LFXIN): now also C12.1, Y1.2
- net at U1.78 (PJ.5_LFXOUT): now also C11.1, Y1.1
- net ADC renamed ADC_DIFF
- net P1.4_PIN_JMP: no longer names the net of J5.5 (Pin_5)
- net P1.4_PIN_JMP: no longer U1.17 (P1.4_TB0.1_UCA0STE_A4_C4)
- new net: C12.2, NT1.2
- new net: C11.2, NT2.2
- new net: NT3.2, U1.76 (AVSS2)
- new net: NT4.2, U1.79 (AVSS1)
- new net ADC_LOAD: U1.17 (P1.4_TB0.1_UCA0STE_A4_C4)
- new net Crystal_GND: NT1.1, NT2.1, NT3.1, NT4.1
- no-connect marks 47 -> 43
