File: energyReplay/energyReplay.kicad_pcb (KiCad board)
At the start: 2 copper layers, 80 x 58 mm, 48 parts, among them J1 Conn_02x07_Odd_Even, J2 Power Select, J3 Conn_01x02_Pin, J4 Conn_01x02_Pin, J5 Conn_02x10_Counter_Clockwise, J6 Conn_01x02_Pin, J7 Conn_01x02_Pin, SW1 SW_Push, SW2 SW_Push, U1 MSP430FR5994IPN, U2 MCP4725xxx-xCH, U3 OPA2387DGKR, U4 TPS613222ADBV, U5 LM66100DCKR

Commit message: 1.1 KiCAD project
Parts:
- added C11: 100n, Capacitor_SMD:C_1206_3216Metric, F.Cu at (93.8, 72.2)
- added C12: 100n, Capacitor_SMD:C_1206_3216Metric, F.Cu at (101.2, 72.2)
- added NT1: NetTie_2, NetTie-0.2mm:NetTie-2_SMD_Pad0.2mm, F.Cu at (101.2, 69.0)
- added NT2: NetTie_2, NetTie-0.2mm:NetTie-2_SMD_Pad0.2mm, F.Cu at (93.8, 69.0)
- added NT3: NetTie_2, NetTie-0.2mm:NetTie-2_SMD_Pad0.2mm, F.Cu at (98.0, 77.0)
- added NT4: NetTie_2, NetTie-0.2mm:NetTie-2_SMD_Pad0.2mm, F.Cu at (96.5, 77.0)
- added Y1: Crystal, MS1V-T1K:XTAL_MS1V-T1K-32.768KHZ-12.5PF-20PPM-TA-QC, F.Cu at (97.2, 70.2)
- moved C3 11.5 mm to (107.5, 70.2)
- moved C1 3.22 mm to (104.5, 98.5)
- moved C2 1.80 mm to (107.5, 74.0)
Connections:
- net ADC renamed ADC_DIFF
- J5 pad 12: unconnected-(J5-Pin_12-Pad12) -> GND
- J5 pad 13: unconnected-(J5-Pin_13-Pad13) -> GND
- J5 pad 14: unconnected-(J5-Pin_14-Pad14) -> GND
- J5 pad 5: /Control/P1.4_PIN_JMP -> unconnected-(J5-Pin_5-Pad5)
- J6 pad 2: Net-(J6-Pin_2) -> ADC_LOAD
- R13 pad 2: Net-(J6-Pin_2) -> ADC_LOAD
- R15 pad 1: Net-(J6-Pin_2) -> ADC_LOAD
- U1 pad 17: /Control/P1.4_PIN_JMP -> ADC_LOAD
- U1 pad 76: GND -> Net-(U1-AVSS2)
- U1 pad 77: unconnected-(U1-PJ.4_LFXIN-Pad77) -> Net-(U1-PJ.4_LFXIN)
- U1 pad 78: unconnected-(U1-PJ.5_LFXOUT-Pad78) -> Net-(U1-PJ.5_LFXOUT)
- U1 pad 79: GND -> Net-(U1-AVSS1)
Routing:
- net ADC_LOAD: track 0.00 -> 68.3 mm, vias 0 -> 6
- net /Control/P1.4_PIN_JMP: track 41.4 -> 0.00 mm, vias 2 -> 0
- net /Control/P2.3_PIN_JMP: track 35.0 -> 69.5 mm
- net /Control/P2.7_PIN_JMP: track 36.1 -> 64.6 mm, vias 2 -> 1
- net /Control/P2.1_PIN_JMP: track 60.3 -> 32.8 mm, vias 5 -> 3
- net /Control/LED1: track 50.8 -> 26.2 mm, vias 4 -> 2
- net Net-(J6-Pin_2): track 9.76 -> 0.00 mm
- net Net-(U1-PJ.4_LFXIN): track 0.00 -> 7.90 mm
- net +3V3: track 260.0 -> 252.2 mm
- net Net-(U1-PJ.5_LFXOUT): track 0.00 -> 7.38 mm
- net ADC_DIFF: track 47.4 -> 53.6 mm
- net /Control/P2.4_PIN_JMP: track 32.6 -> 36.8 mm
- net /Control/P1.5_PIN_JMP: track 21.8 -> 25.9 mm
- net /Control/Crystal_GND: track 0.00 -> 3.87 mm, vias 0 -> 4
- net GND: track 88.9 -> 91.4 mm, vias 14 -> 15
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- added copper zone on B.Cu, net /Control/Crystal_GND
Other:
- board text added: "3V3"
- board text added: "DBG | 3V3"
- board text added: "Energy Replay V1.1 FoRTE Research Virginia Tech"
- board text removed: "DBG | Vin"
- board text removed: "Energy Replay V1.0 FoRTE Research Virginia Tech"
- board text removed: "P1.4"
- board text removed: "Vin"

Commit message: 1.2 KiCAD project and code
Parts:
- added R18: 820k, Resistor_SMD:R_1206_3216Metric, F.Cu at (135.8, 94.0)
- added R19: 820k, Resistor_SMD:R_1206_3216Metric, F.Cu at (138.5, 94.0)
- moved R13 4.74 mm to (137.5, 89.8), turned to 0 degrees
- moved C10 1.03 mm to (132.5, 90.0)
- moved C9 1.03 mm to (132.5, 86.0)
Connections:
- J6 pad 2: ADC_LOAD -> Net-(J6-Pin_2)
- R13 pad 2: ADC_LOAD -> Net-(J6-Pin_2)
- R15 pad 1: ADC_LOAD -> Net-(J6-Pin_2)
Routing:
- net Net-(J6-Pin_2): track 0.00 -> 17.7 mm
- net ADC_LOAD: track 68.3 -> 72.1 mm
- net GND: track 91.4 -> 92.9 mm, vias 15 -> 16
- net +5V: track 21.1 -> 20.5 mm
Other:
- board text added: "Energy Replay V1.2 FoRTE Research Virginia Tech"
- board text removed: "Energy Replay V1.1 FoRTE Research Virginia Tech"
