File: energyReplay/output.kicad_sch (KiCad schematic)
At the start: 24 parts, among them J6 Conn_01x02_Pin, J7 Conn_01x02_Pin, U2 MCP4725xxx-xCH, U3 OPA2387DGKR, U4 TPS613222ADBV, U5 LM66100DCKR

Commit message: 1.1 KiCAD project
Connections:
- net ADC_LOAD: now reaches J6.2 (Pin_2), R13.2, R15.1
- net ADC renamed ADC_DIFF
Changed lines of the file:
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@@
   (title_block
     (title "Power/Measurement")
-    (date "2024-01-22")
-    (rev "0")
+    (date "2024-08-16")
+    (rev "1")
   )
   (junction (at 167.64 76.2) (diameter 0) (color 0 0 0 0)
@@
     (stroke (width 0) (type default))
   )
+  (wire (pts (xy 129.54 31.75) (xy 130.81 31.75))
+    (stroke (width 0) (type default))
+  )
   (wire (pts (xy 33.02 90.17) (xy 34.29 90.17))
     (stroke (width 0) (type default))
@@
     (stroke (width 0) (type default))
   )
+  (wire (pts (xy 129.54 43.18) (xy 129.54 31.75))
+    (stroke (width 0) (type default))
+  )
   (wire (pts (xy 129.54 58.42) (xy 129.54 60.96))
     (stroke (width 0) (type default))
@@
   (text "150x Diff amp for current sense" (at 138.43 95.25 0)
     (effects (font (size 1.27 1.27)) (justify left bottom))
+  )
+  (global_label "ADC_LOAD" (shape input) (at 130.81 31.75 0) (fields_autoplaced)
+    (effects (font (size 1.27 1.27)) (justify left))
+    (property "Intersheetrefs" "${INTERSHEET_REFS}" (at 143.1086 31.75 0)
+      (effects (font (size 1.27 1.27)) (justify left) hide)
+    )
   )
   (global_label "SDA" (shape input) (at 25.4 40.64 180) (fields_autoplaced)
@@
     )
   )
-  (global_label "ADC" (shape input) (at 171.45 76.2 0) (fields_autoplaced)
+  (global_label "ADC_DIFF" (shape input) (at 171.45 76.2 0) (fields_autoplaced)
     (effects (font (size 1.27 1.27)) (justify left))
-    (property "Intersheetrefs" "${INTERSHEET_REFS}" (at 178.0638 76.2 0)
+    (property "Intersheetrefs" "${INTERSHEET_REFS}" (at 183.0834 76.2 0)
       (effects (font (size 1.27 1.27)) (justify left) hide)
     )

Commit message: 1.2 KiCAD project and code
Parts:
- added R18, R19: 820k, Resistor_SMD:R_1206_3216Metric, symbol Device:R
Connections:
- net ADC_LOAD: now also R18.1, R19.1; no longer J6.2 (Pin_2), R13.2, R15.1
- net GND: now also R18.2
- new net: J6.2 (Pin_2), R13.2, R15.1, R19.2
Other:
- moved on the sheet: J6, R13, R14, R15, R16, R17, U3A
